File: KiCad/BodyTempSensor.kicad_sch (KiCad schematic)
At the start: 71 parts, among them IC1 MAX30208CLB+T, J1 USB_C_Receptacle_USB2.0, J2 BAT, J3 TC2030, Q1 NMOS, U1 nRF52840, U2 USBLC6-2SC6, U3 MCP73833-xxx-UN, U4 TLV62568DBVR, U5 MCP6001-OT, U6 LSM6DSO32TR, Y1 32MHz

Commit message: Changed temp sensor, added components and created a general layout design
Parts:
- removed J2: BAT, Connector_PinSocket_2.54mm:PinSocket_1x02_P2.54mm_Vertical, symbol Connector_Generic:Conn_01x02
- removed J3: TC2030, Connector:Tag-Connect_TC2030-IDC-NL_2x03_P1.27mm_Vertical, symbol Connector:TC2030
- added C21: 100n, Capacitor_SMD:C_0504_1310Metric_Pad0.83x1.28mm_HandSolder, symbol Device:C
- added C22, C23: 100n, Capacitor_SMD:C_0402_1005Metric_Pad0.74x0.62mm_HandSolder, symbol Device:C
- added IC2: MAX30208CLB+T, PCB_Lib_ItsNotDaan:MAX30208CLBT, symbol LibLoader:MAX30208CLB+T
- added IC3, IC4: TMP117MAIDRVT, LibLoader:SON65P200X200X80-7N, symbol PCB_Lib_ItsNotDaan:TMP117MAIDRVT
- added J2: TC2030, Connector:Tag-Connect_TC2030-IDC-NL_2x03_P1.27mm_Vertical, symbol Connector:TC2030
- added J3: BAT, Connector_PinSocket_2.54mm:PinSocket_1x02_P2.54mm_Vertical, symbol Connector_Generic:Conn_01x02
- added J4, J7: 52271-0479, LibLoader:522710479, symbol PCB_Lib_ItsNotDaan:52271-0479
- added J5: Conn_01x10, Connector_PinHeader_2.54mm:PinHeader_1x10_P2.54mm_Vertical, symbol Connector_Generic:Conn_01x10
- added J6: Conn_02x05_Odd_Even, Connector_PinSocket_2.54mm:PinSocket_2x05_P2.54mm_Vertical, symbol Connector_Generic:Conn_02x05_Odd_Even
- added Q2: NMOS, symbol Simulation_SPICE:NMOS
- added R25: 10k, Resistor_SMD:R_0402_1005Metric_Pad0.72x0.64mm_HandSolder, symbol Device:R
- added R26, R27: 5k1, Resistor_SMD:R_0402_1005Metric_Pad0.72x0.64mm_HandSolder, symbol Device:R
- added R28: 180k, Resistor_SMD:R_0402_1005Metric_Pad0.72x0.64mm_HandSolder, symbol Device:R
- C10: value 12p -> 100n; LCSC PART # (none) -> C361203; Manufacturer_Name (none) -> YAGEO; Manufacturer_Part_Number (none) -> C1005X5R1E104KT000E
- C13, IC1, R15, R16, R7, RST1: now not fitted; now left out of the parts list
- C15: footprint Capacitor_SMD:C_0402_1005Metric_Pad0.74x0.62mm_HandSolder -> Capacitor_SMD:C_0504_1310Metric_Pad0.83x1.28mm_HandSolder; now not fitted; now left out of the parts list
- C16: value 4u7 -> 100n; footprint Capacitor_SMD:C_0402_1005Metric_Pad0.74x0.62mm_HandSolder -> Capacitor_SMD:C_0504_1310Metric_Pad0.83x1.28mm_HandSolder; LCSC PART # C82453 -> C361203; Manufacturer_Name Murata Electronics -> YAGEO; Manufacturer_Part_Number GRM155R60J475ME47D -> C1005X5R1E104KT000E; now not fitted; now left out of the parts list
- C17: value 270n -> 4u7; LCSC PART # (none) -> C82453; Manufacturer_Name (none) -> Murata Electronics; Manufacturer_Part_Number (none) -> GRM155R60J475ME47D
- C18: value 10u -> 390n; LCSC PART # C2992625 -> (none); Manufacturer_Name FH (Guangdong Fenghua Advanced Tech) -> (none); Manufacturer_Part_Number 0402X106M100CT -> (none)
- C19: value 100n -> 10u; footprint Capacitor_SMD:C_1206_3216Metric -> Capacitor_SMD:C_0402_1005Metric_Pad0.74x0.62mm_HandSolder; LCSC PART # (none) -> C2992625; Manufacturer_Name (none) -> FH (Guangdong Fenghua Advanced Tech); Manufacturer_Part_Number (none) -> 0402X106M100CT; now fitted; now in the parts list
- C2: value 100n -> 1u; footprint Capacitor_SMD:C_0402_1005Metric_Pad0.74x0.62mm_HandSolder -> Capacitor_SMD:C_0504_1310Metric_Pad0.83x1.28mm_HandSolder; LCSC PART # C361203 -> (none); Manufacturer_Name YAGEO -> (none); Manufacturer_Part_Number C1005X5R1E104KT000E -> (none)
- C20: footprint Capacitor_SMD:C_1206_3216Metric -> Capacitor_SMD:C_0504_1310Metric_Pad0.83x1.28mm_HandSolder
- C3: value 1u -> 100n; footprint Capacitor_SMD:C_1206_3216Metric -> Capacitor_SMD:C_0402_1005Metric_Pad0.74x0.62mm_HandSolder; LCSC PART # (none) -> C361203; Manufacturer_Name (none) -> YAGEO; Manufacturer_Part_Number (none) -> C1005X5R1E104KT000E
- C4: value 100n -> 0p8; LCSC PART # C361203 -> (none); Manufacturer_Name YAGEO -> (none); Manufacturer_Part_Number C1005X5R1E104KT000E -> (none)
- C5: value 0p8 -> 100n; footprint Capacitor_SMD:C_0504_1310Metric_Pad0.83x1.28mm_HandSolder -> Capacitor_SMD:C_0402_1005Metric_Pad0.74x0.62mm_HandSolder; LCSC PART # (none) -> C361203; Manufacturer_Name (none) -> YAGEO; Manufacturer_Part_Number (none) -> C1005X5R1E104KT000E
- C8: value 100n -> 0p5; LCSC PART # C361203 -> (none); Manufacturer_Name YAGEO -> (none); Manufacturer_Part_Number C1005X5R1E104KT000E -> (none)
- C9: value 0p5 -> 12p; footprint Capacitor_SMD:C_0504_1310Metric_Pad0.83x1.28mm_HandSolder -> Capacitor_SMD:C_0402_1005Metric_Pad0.74x0.62mm_HandSolder
- R11: value 330k -> 68k
- R17: value 450k -> 82k; LCSC PART # C5159688 -> (none); Manufacturer_Name FOJAN -> (none); Manufacturer_Part_Number FRC0402F4503TS -> (none)
- R18: value 100k -> 450k; LCSC PART # C705662 -> C5159688; Manufacturer_Name YAGEO -> FOJAN; Manufacturer_Part_Number RT0402CRE07100KL -> FRC0402F4503TS
- R19: value 120k -> 100k; LCSC PART # (none) -> C705662; Manufacturer_Name (none) -> YAGEO; Manufacturer_Part_Number (none) -> RT0402CRE07100KL
- R20: footprint Resistor_SMD:R_1206_3216Metric -> Resistor_SMD:R_0402_1005Metric_Pad0.72x0.64mm_HandSolder; LCSC PART # (none) -> C163810; Manufacturer_Name (none) -> Walsin Tech Corp; Manufacturer_Part_Number (none) -> WR04X1002FTL; now fitted; now in the parts list
- R21: value 47k -> 180k
- R22: value 180k -> 47k
- R23: value 10k -> 180k; LCSC PART # C163810 -> (none); Manufacturer_Name Walsin Tech Corp -> (none); Manufacturer_Part_Number WR04X1002FTL -> (none)
- R24: value 180k -> 10k; footprint Resistor_SMD:R_0402_1005Metric_Pad0.72x0.64mm_HandSolder -> Resistor_SMD:R_1206_3216Metric; now not fitted; now left out of the parts list
- R4, R5, R6, R9: footprint Resistor_SMD:R_1206_3216Metric -> Resistor_SMD:R_0402_1005Metric_Pad0.72x0.64mm_HandSolder
Connections:
- net +1V8: now also R24.1, C21.2; no longer C19.2, R20.1
- net +3V3: now also C10.1, C15.1, C16.1, C19.1, C3.1, C5.1, IC1.1 (VDD_1), IC1.2 (VDD_2), IC1.3 (VDD_3), R18.1, C22.1, C23.1, IC2.1 (VDD_1), IC2.10 (GPIO0), IC2.2 (VDD_2), IC2.3 (VDD_3), IC3.4 (ADD0), IC3.5 (V+), IC4.5 (V+), J2.1, J4.1, J5.1 (Pin_1), J6.1 (Pin_1), J7.1, R26.1, R27.1; no longer C18.1, C2.1, C4.1, C8.1, R17.1
- net Earth: now also C17.2, C19.2, C2.1, C3.2, IC1.10 (GPIO0), IC1.7 (GPIO1), R19.2, R21.2, C21.1, C22.2, C23.2, IC2.4 (GND_1), IC2.5 (GND_2), IC2.6 (GND_3), IC2.7 (GPIO1), IC3.2 (GND), IC4.2 (GND), IC4.4 (ADD0), J2.3, J2.5, J3.1 (Pin_1), J4.4, J4.MP1, J4.MP2, J5.10 (Pin_10), J6.3 (Pin_3), J6.5 (Pin_5), J7.4, J7.MP1, J7.MP2, Q2.3 (S), R28.2; no longer C18.2, C19.1, C2.2, C3.1, R18.2, R24.2, U5.2 (V-)
- net OSC_OUT: now also C9.1; no longer C10.1
- net P0.02: now also C18.2, R17.2, J5.2 (Pin_2); no longer C17.2, R19.2
- net P0.03: now also J5.3 (Pin_3)
- net P0.13: now also J5.4 (Pin_4)
- net P0.15: now also R22.2, R23.1, J5.5 (Pin_5); no longer R21.2, R22.1
- net P0.16: now also R20.1, J5.6 (Pin_6); no longer R23.1
- net P0.17/SDA: now also IC2.8 (SDA), IC3.6 (SDA), IC4.6 (SDA), J4.2, J5.7 (Pin_7), J7.2, R27.2
- net P0.19/SCL: now also IC2.9 (SCL), IC3.1 (SCL), IC4.1 (SCL), J4.3, J5.8 (Pin_8), J7.3, R26.2
- net RF: now also C4.1; no longer C5.1
- net RF2: now also C8.1; no longer C9.1
- net VBAT: now also C17.1, R22.1, J3.2 (Pin_2); no longer C16.1, R21.1
- net VBUS: now also C2.2; no longer C3.2
- net nRF_RESET: now also J2.6
- net nRF_SWD_CLK: now also J2.4, J6.4 (Pin_4)
- net nRF_SWD_DIO: now also J2.2, J6.2 (Pin_2)
- net at H2.1, U5.4 (-): now also C18.1, R17.1; no longer C17.1, R19.1
- net at Q1.1 (D): now also R23.2; no longer R22.2
- net at U6.12 (CS): now also R24.2; no longer R20.2
- new net: R18.2, R19.1, U4.5 (FB)
- new net: Q1.2 (G), R20.2, R21.1
- new net: Q2.2 (G), R25.2, R28.1
- new net AMP_1: Q2.1 (D), U5.2 (V-)
- new net P0.04: R25.1
- no-connect marks 10 -> 17
Other:
- note added: "1001000x"
- note added: "1001001x"
- note added: "Current: Stand-By: 0.5uA Operating: 22uA max: 135uA"
- note added: "Funct: SWD the nRF target. Debug, flash and check on it. Using the nRF52840-DK dev board as a bootloader flasher."
- note added: "I2C = 0x0"
- note added: "I2C = 0x1"
- note added: "LX FFC 4P 1.0mm 20CM"
- note added: "Links:"
- note added: "MOLEX 522710479"
- note added: "TC2030 (Expensive)"
- note added: "TMP117MAIDRVR"
- note added: "https://www.ti.com/lit/ug/tidudw4b/tidudw4b.pdf?ts=1779587732925"
- note removed: "0,52->1,354v 1,65V − 0,296V = 1,354V 1,65V − 1,131V = 0,519V"

Commit message: Add Bill of Materials (BOM) for Body Temperature Sensor project
Parts:
- removed C15, C16, C20, C21: 100n, Capacitor_SMD:C_0504_1310Metric_Pad0.83x1.28mm_HandSolder, symbol Device:C
- removed IC1, IC2: MAX30208CLB+T, PCB_Lib_ItsNotDaan:MAX30208CLBT, symbol LibLoader:MAX30208CLB+T
- removed J2: TC2030, Connector:Tag-Connect_TC2030-IDC-NL_2x03_P1.27mm_Vertical, symbol Connector:TC2030
- removed J4, J7: 52271-0479, LibLoader:522710479, symbol PCB_Lib_ItsNotDaan:52271-0479
- removed J5: Conn_01x10, Connector_PinHeader_2.54mm:PinHeader_1x10_P2.54mm_Vertical, symbol Connector_Generic:Conn_01x10
- removed R15, R16: 5k1, Resistor_SMD:R_0402_1005Metric_Pad0.72x0.64mm_HandSolder, symbol Device:R
- removed R24: 10k, Resistor_SMD:R_1206_3216Metric, symbol Device:R
- removed U1: nRF52840, Package_DFN_QFN:Nordic_AQFN-73-1EP_7x7mm_P0.5mm, symbol MCU_Nordic:nRF52840
- removed U6: LSM6DSO32TR, PCB_Lib_ItsNotDaan_KiCad:LGA-14_3x2.5mm_P0.5mm_LayoutBorder3x4y, symbol Sensor_Motion:LSM6DS3
- added C24, C25, C26: 100n, Capacitor_SMD:C_0402_1005Metric_Pad0.74x0.62mm_HandSolder, symbol Device:C
- added C27: 10n, Capacitor_SMD:C_0402_1005Metric_Pad0.74x0.62mm_HandSolder, symbol Device:C
- added C28, C30: 2u2, Capacitor_SMD:C_0402_1005Metric_Pad0.74x0.62mm_HandSolder, symbol Device:C
- added C29: 2n2, Capacitor_SMD:C_0402_1005Metric_Pad0.74x0.62mm_HandSolder, symbol Device:C
- added IC5, IC6: TMP117MAIDRVT, LibLoader:SON65P200X200X80-7N, symbol PCB_Lib_ItsNotDaan:TMP117MAIDRVT
- added IC7: NRF54L15-QFAA-R, LibLoader:QFN40P600X600X95-49N, symbol LibLoader:NRF54L15-QFAA-R
- added L3: 2.7nH, Inductor_SMD:L_0201_0603Metric, symbol Device:L
- added L4: 3.5nH, Inductor_SMD:L_0201_0603Metric, symbol Device:L
- added L5: 4u7, Inductor_SMD:L_0201_0603Metric, symbol Device:L
- C4: value 0p8 -> 1p5
- C8: value 0p5 -> 2p
- IC3: value TMP117MAIDRVT -> TMP117MAIDRVR
- J6: footprint Connector_PinSocket_2.54mm:PinSocket_2x05_P2.54mm_Vertical -> Connector_PinHeader_1.27mm:PinHeader_2x05_P1.27mm_Vertical
- L1: value 4n7 -> 3.5nH; footprint Inductor_SMD:L_0402_1005Metric_Pad0.77x0.64mm_HandSolder -> Inductor_SMD:L_0201_0603Metric; Manufacturer_Part_Number (none) -> LQP03HQ3N5B02
Connections:
- net +3V3: now also C24.1, C25.1, C26.1, IC5.5 (V+), IC6.5 (V+), IC7.10 (VDD_1), IC7.22 (VDD_2), IC7.36 (VDD_3), IC7.47 (VDD_4), IC7.48 (VDD_5)
- net Earth: now also C24.2, C25.2, C26.2, C27.2, C28.2, C29.2, C30.2, IC5.2 (GND), IC6.2 (GND), IC7.32 (VSS_PA), IC7.44 (VSS), IC7.49 (EP)
- net OSC_IN: now also IC7.34 (XC1)
- net OSC_OUT: now also IC7.35 (XC2)
- net P0.17/SDA: now also IC5.4 (ADD0), IC5.6 (SDA), IC6.6 (SDA)
- net P0.19/SCL: now also IC5.1 (SCL), IC6.1 (SCL), IC6.4 (ADD0)
- net RF: now also IC7.31 (ANT), L3.1; no longer C4.1, L1.1
- net RF2: now also L4.2; no longer C8.1, L1.2
- net nRF_RESET: now also J6.10 (Pin_10), IC7.30 (NRESET)
- net nRF_SWD_CLK: now also IC7.26 (SWDCLK)
- net nRF_SWD_DIO: now also IC7.25 (SWDIO)
- net P0.02 renamed IO_IMP_OUT
- net P0.03 renamed IO_IMP_IN
- net P0.04 renamed IO_IMP_PWR
- net P0.13 renamed IO_RGB
- net P0.14 renamed IO_BTN_ACT
- net P0.15 renamed IO_BAT_MEAS
- net P0.16 renamed IO_BAT_MEAS_ON
- new net: C4.1, L1.1, L3.2
- new net: C30.1, IC7.45 (DECD), L5.1
- new net: IC7.46 (DCC), L5.2
- new net: C8.1, L1.2, L4.1
- new net: C28.1, C29.1, IC7.33 (DECRF)
- new net: C27.1, IC7.43 (DECA)
- no-connect marks 17 -> 15
Other:
- note added: "1001010x"
- note added: "1001011x"
- note removed: "Current: Stand-By: 0.5uA Operating: 67uA max: 100uA"
- note removed: "Funct: Interrupt for movement."
- note removed: "Funct: SWD the nRF target. Debug, flash and check on it."
- note removed: "Gyroscope"
- note removed: "I2C = 0x0"
- note removed: "I2C = 0x1"
- note removed: "LSM6DSO32TR"
- note removed: "LX FFC 4P 1.0mm 20CM"
- note removed: "MAX30208CLB+T"
- note removed: "MOLEX 522710479"
- note removed: "TC2030"
- note removed: "https://www.sparkfun.com/products/18020"
- moved on the sheet: ACT1, ANT1, C1, C10, C11, C12, C13, C14, C17, C18, C19, C22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
